Commit message: check of already implemented code, still need to check docs

File: urdf/robot.xacro (robot description, xacro)
@@ -40,5 +40,5 @@
     <color rgba="1.0 1.0 1.0 1.0"/>
   </material>
-	  <link name="link_chassis">
+	<link name="link_chassis">
     <!-- pose and inertial -->
     <pose>0 0 0.1 0 0 0</pose>
@@ -51,5 +51,5 @@
     <collision name="collision_chassis">
       <geometry>
-        <box size="0.5 0.3 0.07"/>
+        <box size="0.5 0.3 0.1"/>
       </geometry>
     </collision>
@@ -57,7 +57,7 @@
       <origin rpy="0 0 0" xyz="0 0 0"/>
       <geometry>
-        <box size="0.5 0.3 0.07"/>
-      </geometry>
-      <material name="blue"/>
+        <box size="0.5 0.3 0.1"/>
+      </geometry>
+      <material name="orange"/>
     </visual>
     <!-- caster front -->
@@ -75,5 +75,6 @@
     </visual>
   </link>
-   <link name="link_right_wheel">
+  <!-- wheels -->
+  <link name="link_right_wheel">
     <xacro:default_inertial mass="0.2"/>
     <collision name="link_right_wheel_collision">
@@ -115,19 +116,65 @@
     <joint_properties damping="1.0" friction="1.0"/>
   </joint>
+  <!-- neck and head -->
+  <link name="link_neck">
+    <xacro:default_inertial mass="0.5"/>
+    <collision name="link_neck_collision">
+      <origin rpy="0 0 0" xyz="0.1 0 0.05"/>
+      <geometry>
+        <cylinder length="0.1" radius="0.05"/>
+      </geometry>
+    </collision>
+    <visual name="link_neck_visual">
+      <origin rpy="0 0 0" xyz="0.1 0 0.05"/>
+      <geometry>
+        <cylinder length="0.1" radius="0.05"/>
+      </geometry>
+      <material name="orange"/>
+    </visual>
+  </link>
+  <link name="link_head">
+    <xacro:default_inertial mass="0.5"/>
+    <collision name="link_head_collision">
+      <origin rpy="0 0 0" xyz="0.15 0 0.15"/>
+      <geometry>
+        <box size= "0.15 0.2 0.15"/>
+      </geometry>
+    </collision>
+    <visual name="link_head_visual">
+      <origin rpy="0 0 0" xyz="0.15 0 0.15"/>
+      <geometry>
+        <box size= "0.15 0.2 0.15"/>
+      </geometry>
+      <material name="orange"/>
+    </visual>
+  </link>
+  <joint name="joint_neck" type="fixed">
+    <axis xyz="0 1 0" />
+	  <origin xyz="0.1 0 0.05" rpy="0 0 0"/>
+    <child link="link_neck"/>
+    <parent link="link_chassis"/>
+  </joint>
+  <joint name="joint_head" type="revolute">
+    <origin rpy="0 0 0" xyz="0 0 0"/>
+    <child link="link_head"/>
+    <parent link="link_neck"/>
+    <axis xyz="0 0 1"/>
+    <limit effort="1000.0" lower="-1.57" upper="1.57" velocity="0.1"/>/>
+    <joint_properties damping="1.0" friction="1.0"/>
+  </joint>
+  <!-- camera -->
   <link name="camera_link">
 	    <collision>
-	      <origin xyz="0 0 0.025" rpy="0 0 0"/>
+	      <origin xyz="0.025 0 0.15" rpy="0 0 0"/>
 	      <geometry>
-		<box size="0.05 0.05 0.05"/>
+		      <box size="0.05 0.05 0.05"/>
 	      </geometry>
 	    </collision>
 	    <visual>
-	      <origin xyz="0 0 0.025" rpy="0 0 0"/>
+	      <origin xyz="0.025 0 0.15" rpy="0 0 0"/>
 	      <geometry>
-		<box size="0.05 0.05 0.05"/>
+		      <box size="0.05 0.05 0.05"/>
 	      </geometry>
-	      <material name="red">
-		<color rgba="1 0 0 1"/>
-	      </material>
+	      <material name="grey"/>
 	    </visual>
 	    <inertial>
@@ -139,7 +186,17 @@
   <joint name="camera_joint" type="fixed">
 	    <axis xyz="0 1 0" />
-	    <origin xyz="0.23 0 0.0" rpy="0 0 0"/>
-	    <parent link="link_chassis"/>
-	    <child link="camera_link"/>
-	 </joint>
+	    <origin xyz="0.15 0 0.0" rpy="0 0 0"/>
+      <child link="camera_link"/>
+	    <parent link="link_head"/>
+	</joint>
+  <transmission name="joint_head_trans">
+	  <type>transmission_interface/SimpleTransmission</type>
+	  <joint name="joint_head">
+		<hardwareInterface>hardware_interface/EffortJointInterface</hardwareInterface>
+	</joint>
+	<actuator name="motor1">
+		<hardwareInterface>hardware_interface/EffortJointInterface</hardwareInterface>
+		<mechanicalInterface>1</mechanicalInterface>
+	</actuator>
+  </transmission>
 </robot>
